File: PCB_V3_PADAUK/pcb/pcb.sch (KiCad schematic (older format))
At the start: 41 parts, among them J1 FLUSH_SWITCH, J2 ISP, J3 BATTERY, J4 SOLENOID, J5 BUZZER_CONN, J6 L_DETECT, J7 Programming Connector, Q1 DMG2301L, Q2 BC817, Q3 BC817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

Commit message: Add files via upload
Via updated
Parts:
- J7: footprint Connector_PinHeader_2.54mm:PinHeader_2x03_P2.54mm_Vertical -> pcb:PinHeader_2x03_P2.54mm_Vertical
Changed lines of the file:
@@
 F 0 "J7" V 2472 7180 50  0000 L CNN
 F 1 "Programming Connector" V 2563 7180 50  0000 L CNN
-F 2 "Connector_PinHeader_2.54mm:PinHeader_2x03_P2.54mm_Vertical" H 2600 6900 50  0001 C CNN
+F 2 "pcb:PinHeader_2x03_P2.54mm_Vertical" H 2600 6900 50  0001 C CNN
 F 3 "~" H 2600 6900 50  0001 C CNN
 	1    2600 6900
