File: PCB_V3_PADAUK/pcb/pcb.kicad_pcb (KiCad board)
At the start: 2 copper layers, 54.6 x 26.7 mm, 41 parts, among them J1 FLUSH_SWITCH, J3 BATTERY, J4 SOLENOID, J5 BUZZER_CONN, J6 L_DETECT, J7 Programming Connector, Q1 DMG2301L, Q2 BC817, Q3 BC817, Q4 DMG2301L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

Commit message: Add files via upload
Via updated
Parts:
- J7: footprint Connector_PinHeader_2.54mm:PinHeader_2x03_P2.54mm_Vertical -> pcb:PinHeader_2x03_P2.54mm_Vertical
- moved J7 0.23 mm to (104.9, 95.1)
Routing:
- net GND: track 29.4 -> 30.2 mm, vias 63 -> 64
- net +1V8: track 72.6 -> 73.3 mm, vias 3 -> 4
- net Net-(J7-Pad6): track 21.2 -> 21.5 mm, vias 3 -> 4
- net POWER_CONTROL: track 44.7 -> 44.5 mm, vias 2 -> 3
- net XTAL2: track 27.7 -> 27.8 mm, vias 1 -> 2
- net BUZZER: track 20.7 -> 20.6 mm, vias 0 -> 1

Commit message: Add files via upload
Connections:
- J7 pad 6: Net-(J7-Pad6) -> GND
- U1 pad 7: Net-(J7-Pad6) -> GND
Routing:
- net Net-(J7-Pad6): track 21.5 -> 0.00 mm, vias 4 -> 0
- net GND: track 30.2 -> 50.4 mm, vias 64 -> 71
- net L_DETECT: track 21.4 -> 16.1 mm, vias 3 -> 2
- net POWER_CONTROL: track 44.5 -> 45.8 mm
